File: LightStage.sch (KiCad schematic (older format))
At the start: 125 parts, among them J1 Conn_01x02_Male, J10 Conn_01x02_Male, J11 Conn_01x02_Male, J12 Conn_01x02_Male, J13 Conn_01x02_Male, J14 Conn_01x02_Male, J15 Conn_01x02_Male, J17 Conn_01x02_Male, J18 Conn_01x02_Male, J19 Conn_01x02_Male, J2 Conn_01x02_Male, J20 Conn_01x02_Male, J21 Conn_01x02_Male, J22 Conn_01x02_Male, J23 Conn_01x02_Male, J24 Conn_01x02_Male, J25 Conn_01x02_Male, J26 Conn_01x02_Male, J3 Conn_01x02_Male, J4 Conn_01x02_Male, J5 Conn_01x02_Male, J6 Conn_01x02_Male, J7 Conn_01x02_Male, J8 Conn_01x02_Male, J9 Conn_01x02_Male, U1 PCA9685PW, U10 TPS92200D2DDCR, U11 TPS92200D2DDCR, U12 TPS92200D2DDCR, U13 TPS92200D2DDCR, U14 TPS92200D2DDCR, U15 TPS92200D2DDCR, U16 TPS92200D2DDCR, U17 TPS92200D2DDCR, U18 TPS92200D2DDCR, U19 TPS92200D2DDCR, U2 LM78L05ACM_NOPB, U3 TPS92200D2DDCR, U4 TPS92200D2DDCR, U5 TPS92200D2DDCR, U6 TPS92200D2DDCR, U7 TPS92200D2DDCR, U8 TPS92200D2DDCR

Commit message: Light Stage version 2
Light Stage
Parts:
- removed C3: 0.01uF, Capacitor_SMD:C_0402_1005Metric_Pad0.74x0.62mm_HandSolder, symbol Device:C
- removed C37: 0.1uF, Capacitor_SMD:C_1206_3216Metric_Pad1.33x1.80mm_HandSolder, symbol Device:C
- removed C46: 10uF, Capacitor_SMD:C_1206_3216Metric_Pad1.33x1.80mm_HandSolder, symbol Device:C
- removed J1, J10, J11, J12, J13, J14, J15, J17, J18, J19, J2, J20, J21, J22, J23, J24, J25, J26, J3, J4, J5, J6, J8, J9: Conn_01x02_Male, Connector_PinHeader_2.54mm:PinHeader_1x02_P2.54mm_Vertical, symbol Connector:Conn_01x02_Male
- removed R10: 10K, Resistor_SMD:R_0603_1608Metric_Pad0.98x0.95mm_HandSolder, symbol Device:R
- removed R4, R5, R6, R7, R8, R9: 10K, Resistor_SMD:R_0402_1005Metric_Pad0.72x0.64mm_HandSolder, symbol Device:R
- added J1: Conn_02x07_Odd_Even, Connector_PinHeader_2.54mm:PinHeader_2x07_P2.54mm_Vertical_SMD, symbol Connector_Generic:Conn_02x07_Odd_Even
- added J10, J11, J12, J13, J14, J15, J16, J17, J18, J19, J4, J5, J6, J7, J8, J9: (no value), 781710004 Pico-EZmate:781710004, symbol 78171004_Pico-EZmate:781710004
- added J20: 781710004, 781710004 Pico-EZmate:781710004, symbol 78171004_Pico-EZmate:781710004
- added RN1: 4609M-101-103LF, SamacSys_Parts:4609X, symbol LightStage-rescue:4609M-101-103LF-SamacSys_Parts
- D1: footprint LED_SMD:LED_0201_0603Metric_Pad0.64x0.40mm_HandSolder -> LED_SMD:LED_0402_1005Metric_Pad0.77x0.64mm_HandSolder
- J2: renamed from J7; footprint Connector_PinHeader_2.54mm:PinHeader_1x02_P2.54mm_Vertical -> SamacSys_Parts:Molex_26013114
- U1: renamed from U2; footprint LM78L05:LM78L05ACM&slash_NOPB -> footprints:LM78L05ACM&slash_NOPB
- U10: renamed from U11; value TPS92200D2DDCR -> (none)
- U11: renamed from U12; value TPS92200D2DDCR -> (none)
- U12: renamed from U13; value TPS92200D2DDCR -> (none)
- U13: renamed from U14; value TPS92200D2DDCR -> (none)
- U14: renamed from U15; value TPS92200D2DDCR -> (none)
- U15: renamed from U16; value TPS92200D2DDCR -> (none)
- U16: renamed from U17; value TPS92200D2DDCR -> (none)
- U17: renamed from U18; value TPS92200D2DDCR -> (none)
- U18: renamed from U19; value TPS92200D2DDCR -> (none)
- U2: renamed from U7; value TPS92200D2DDCR -> (none)
- U3: renamed from U8; value TPS92200D2DDCR -> (none)
- U5: renamed from U4; value TPS92200D2DDCR -> (none)
- U6: renamed from U5; value TPS92200D2DDCR -> (none)
- U7: renamed from U6; value TPS92200D2DDCR -> (none)
- U8: renamed from U3; value TPS92200D2DDCR -> (none)
- U9: renamed from U10; value TPS92200D2DDCR -> (none)
- renumbered C2 to C1, C11 to C10, C12 to C11, C13 to C12, C5 to C13, C17 to C14, C18 to C15, C19 to C16, C7 to C17, C36 to C18, C9 to C2, C38 to C20, C39 to C21, C40 to C22, C41 to C23, C47 to C25, C48 to C26, C49 to C27, C50 to C28, C51 to C29, C15 to C3, C57 to C30, C58 to C31, C59 to C32, C60 to C33, C61 to C34, C67 to C35, C68 to C36, C69 to C37, C70 to C38, C71 to C39, C1 to C5, C22 to C6, C23 to C7, C26 to C8, C27 to C9, L5 to L1, L11 to L10, L12 to L11, L13 to L12, L14 to L13, L15 to L14, L16 to L15, L17 to L16, L6 to L2, L2 to L3, L3 to L4, L4 to L5, L1 to L6, L8 to L7, L9 to L8, L10 to L9, R18 to R10, R19 to R11, R20 to R12, R21 to R13, R22 to R14, R23 to R15, R24 to R16, R25 to R17, R26 to R18, R27 to R19, R15 to R4, R16 to R5, R12 to R6, R13 to R7, R14 to R8, R11 to R9, U1 to U4
Connections:
- net A0: now also J1.2 (Pin_2), RN1.2
- net A1: now also J1.4 (Pin_4), RN1.3
- net A2: now also J1.6 (Pin_6), RN1.4
- net A3: now also J1.8 (Pin_8), RN1.5
- net A4: now also J1.10 (Pin_10), RN1.6
- net A5: now also J1.12 (Pin_12), RN1.7
- net GND: now also J2.2 (Pin_2), RN1.1
- net OE: now also J1.14 (Pin_14), RN1.8
- net PWM10: now also U4.17 (LED10)
- net PWM11: now also U4.18 (LED11)
- net PWM12: now also U4.19 (LED12)
- net PWM13: now also U4.20 (LED13)
- net PWM14: now also U4.21 (LED14)
- net PWM15: now also U4.22 (LED15)
- net PWM3: no longer U11.2 (DIM)
- net PWM6: now also U4.12 (LED6)
- net PWM7: now also U4.13 (LED7)
- net PWM9: now also U4.16 (LED9)
- net SCL: now also J20.4
- net SDA: now also J20.1
- net VCC: now also J1.1 (Pin_1), J1.11 (Pin_11), J1.13 (Pin_13), J1.3 (Pin_3), J1.5 (Pin_5), J1.7 (Pin_7), J1.9 (Pin_9)
- net n_LED0: now also J19.4
- net n_LED1: now also J16.4
- net n_LED10: now also J9.1
- net n_LED11: now also J6.1
- net n_LED12: now also J7.1
- net n_LED13: now also J8.1
- net n_LED14: now also J4.1
- net n_LED15: now also J5.1
- net n_LED2: now also J17.4
- net n_LED3: now also J18.4
- net n_LED4: now also J13.1
- net n_LED5: now also J14.1
- net n_LED6: now also J15.1
- net n_LED7: now also J10.1
- net n_LED8: now also J11.1
- net n_LED9: now also J12.1
- net p_LED0: now also J19.1
- net p_LED1: now also J16.1
- net p_LED10: now also J9.4
- net p_LED11: now also J6.4
- net p_LED12: now also J7.4
- net p_LED13: now also J8.4
- net p_LED14: now also J4.4
- net p_LED15: now also J5.4
- net p_LED2: now also J17.1
- net p_LED3: now also J18.1
- net p_LED4: now also J13.4
- net p_LED5: now also J14.4
- net p_LED6: now also J15.4
- net p_LED7: now also J10.4
- net p_LED8: now also J11.4
- net p_LED9: now also J12.4
- net PWM8: now reaches U4.15 (LED8)
- net PWM8: now also U11.2 (DIM)
Other:
- moved on the sheet: C1, C6, C8, D1, L1, R1, R2, R3, R4, U1, U2

Commit message: The updated kicad drawings
Parts:
- C5: footprint Capacitor_SMD:C_0402_1005Metric_Pad0.74x0.62mm_HandSolder -> Capacitor_SMD:C_1206_3216Metric_Pad1.33x1.80mm_HandSolder
Changed lines of the file:
@@
 F 0 "C5" H 4215 896 50  0000 L CNN
 F 1 "100uF" H 4215 805 50  0000 L CNN
-F 2 "Capacitor_SMD:C_0402_1005Metric_Pad0.74x0.62mm_HandSolder" H 4138 700 50  0001 C CNN
+F 2 "Capacitor_SMD:C_1206_3216Metric_Pad1.33x1.80mm_HandSolder" H 4138 700 50  0001 C CNN
 F 3 "~" H 4100 850 50  0001 C CNN
 	1    4100 850
